Commit message: fixed setup.py

File: urdf/arm-drone/arm-drone.urdf (robot description, URDF)
Before this commit: robot onshape, 5 links, 4 joints
Links:
- link arm: geometry collision mesh filename=package://arm-drone/urdf/arm-drone/arm.stl; visual mesh filename=package://arm-drone/urdf/arm-drone/arm.stl
- link arm_hinge: geometry collision mesh filename=package://arm-drone/urdf/arm-drone/arm_hinge.stl; visual mesh filename=package://arm-drone/urdf/arm-drone/arm_hinge.stl
- link drone: geometry collision mesh filename=package://arm-drone/urdf/arm-drone/drone.stl; visual mesh filename=package://arm-drone/urdf/arm-drone/drone.stl
